File: first-3k-keypad.kicad_pcb (KiCad board)
At the start: 2 copper layers, 57.1 x 71.4 mm, 24 parts, among them SW1 SW_Push, U1 ATmega32U4-AU, Y1 16MHz

Commit message: Minor Edits
Routing:
- net Net-(D2-Pad2): track 0.00 -> 6.62 mm
Changed lines of the file:
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@@
     (thickness 1.6)
     (drawings 9)
-    (tracks 172)
+    (tracks 173)
     (zones 0)
     (modules 24)
@@
     (0 F.Cu signal)
     (31 B.Cu signal)
-    (32 B.Adhes user)
-    (33 F.Adhes user)
-    (34 B.Paste user)
-    (35 F.Paste user)
-    (36 B.SilkS user)
-    (37 F.SilkS user)
-    (38 B.Mask user)
-    (39 F.Mask user)
-    (40 Dwgs.User user)
-    (41 Cmts.User user)
-    (42 Eco1.User user)
-    (43 Eco2.User user)
-    (44 Edge.Cuts user)
-    (45 Margin user)
-    (46 B.CrtYd user)
-    (47 F.CrtYd user)
-    (48 B.Fab user)
-    (49 F.Fab user)
+    (32 B.Adhes user hide)
+    (33 F.Adhes user hide)
+    (34 B.Paste user hide)
+    (35 F.Paste user hide)
+    (36 B.SilkS user hide)
+    (37 F.SilkS user hide)
+    (38 B.Mask user hide)
+    (39 F.Mask user hide)
+    (40 Dwgs.User user hide)
+    (41 Cmts.User user hide)
+    (42 Eco1.User user hide)
+    (43 Eco2.User user hide)
+    (44 Edge.Cuts user hide)
+    (45 Margin user hide)
+    (46 B.CrtYd user hide)
+    (47 F.CrtYd user hide)
+    (48 B.Fab user hide)
+    (49 F.Fab user hide)
   )
   (setup
@@
   (segment (start 132.97 103.125) (end 129.54 99.695) (width 0.254) (layer F.Cu) (net 6))
   (segment (start 134.9375 103.125) (end 132.97 103.125) (width 0.254) (layer F.Cu) (net 6))
+  (segment (start 115.0335 122.175) (end 115.8875 122.175) (width 0.254) (layer F.Cu) (net 7))
+  (segment (start 112.1835 119.325) (end 115.0335 122.175) (width 0.254) (layer F.Cu) (net 7))
+  (segment (start 110.45 119.325) (end 112.1835 119.325) (width 0.254) (layer F.Cu) (net 7))
   (segment (start 130.12 119.325) (end 129.5 119.325) (width 0.254) (layer F.Cu) (net 9))
   (segment (start 132.97 122.175) (end 130.12 119.325) (width 0.254) (layer F.Cu) (net 9))
@@
   (segment (start 119.853001 113.884245) (end 119.853001 146.659499) (width 0.381) (layer B.Cu) (net 10))
   (segment (start 110.743756 104.775) (end 119.853001 113.884245) (width 0.381) (layer B.Cu) (net 10))
-  (via (at 123.825 103.98125) (size 0.8) (drill 0.4) (layers F.Cu B.Cu) (net 11))
-  (segment (start 123.19 102.235) (end 123.19 103.34625) (width 0.254) (layer F.Cu) (net 11))
-  (segment (start 123.19 103.34625) (end 123.825 103.98125) (width 0.254) (layer F.Cu) (net 11))
   (via (at 124.5 119.825) (size 0.8) (drill 0.4) (layers F.Cu B.Cu) (net 11))
-  (segment (start 123.825 103.98125) (end 124.5 104.65625) (width 0.254) (layer B.Cu) (net 11))
-  (segment (start 124.5 104.65625) (end 124.5 119.825) (width 0.254) (layer B.Cu) (net 11))
+  (segment (start 124.5 103.545) (end 123.19 102.235) (width 0.254) (layer B.Cu) (net 11))
+  (segment (start 124.5 119.825) (end 124.5 103.545) (width 0.254) (layer B.Cu) (net 11))
+  (via (at 123.19 102.235) (size 0.8) (drill 0.4) (layers F.Cu B.Cu) (net 11))
   (segment (start 115.8875 124.771) (end 115.8875 125.475) (width 0.254) (layer F.Cu) (net 12))
   (segment (start 112.4015 121.285) (end 115.8875 124.771) (width 0.254) (layer F.Cu) (net 12))
@@
   (via (at 108.74375 104.775) (size 0.8) (drill 0.4) (layers F.Cu B.Cu) (net 15))
   (segment (start 108.74375 101.3375) (end 108.74375 104.775) (width 0.254) (layer F.Cu) (net 15))
-  (via (at 111.91875 135.73125) (size 0.8) (drill 0.4) (layers F.Cu B.Cu) (net 15))
-  (segment (start 111.91875 124.358816) (end 111.91875 135.73125) (width 0.254) (layer B.Cu) (net 15))
   (segment (start 108.74375 104.775) (end 108.74375 121.183816) (width 0.254) (layer B.Cu) (net 15))
-  (segment (start 108.74375 121.183816) (end 111.91875 124.358816) (width 0.254) (layer B.Cu) (net 15))
   (segment (start 119.20625 135.73125) (end 120.79375 137.31875) (width 0.254) (layer F.Cu) (net 15))
-  (segment (start 111.91875 135.73125) (end 119.20625 135.73125) (width 0.254) (layer F.Cu) (net 15))
+  (via (at 111.125 135.73125) (size 0.8) (drill 0.4) (layers F.Cu B.Cu) (net 15))
+  (segment (start 108.74375 121.183816) (end 111.125 123.565066) (width 0.254) (layer B.Cu) (net 15))
+  (segment (start 111.125 123.565066) (end 111.125 135.73125) (width 0.254) (layer B.Cu) (net 15))
+  (segment (start 111.125 135.73125) (end 119.20625 135.73125) (width 0.254) (layer F.Cu) (net 15))
   (segment (start 122.304 143.65625) (end 121.3 143.65625) (width 0.254) (layer F.Cu) (net 16))
   (segment (start 123.067477 142.892773) (end 122.304 143.65625) (width 0.254) (layer F.Cu) (net 16))

Commit message: Actually Finished this time
Connections:
- U1 pad 29: Net-(U1-Pad29) -> COL0
- U1 pad 30: Net-(U1-Pad30) -> ROW1
- U1 pad 31: Net-(U1-Pad31) -> COL1
- U1 pad 32: Net-(U1-Pad32) -> COL1
Routing:
- net ROW1: track 0.00 -> 40.5 mm
- net COL1: track 69.8 -> 102.5 mm
- net COL0: track 18.1 -> 49.3 mm, vias 2 -> 3
Changed lines of the file:
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@@
     (thickness 1.6)
     (drawings 9)
-    (tracks 173)
+    (tracks 197)
     (zones 0)
     (modules 24)
-    (nets 47)
+    (nets 43)
   )
   (page A4)
@@
     (solder_mask_min_width 0.25)
     (aux_axis_origin 0 0)
-    (visible_elements FFFFFF7F)
+    (visible_elements 7FFFFFFF)
     (pcbplotparams
       (layerselection 0x010fc_ffffffff)
@@
   (net 24 "Net-(U1-Pad37)")
   (net 25 "Net-(U1-Pad36)")
-  (net 26 "Net-(U1-Pad32)")
-  (net 27 "Net-(U1-Pad31)")
-  (net 28 "Net-(U1-Pad30)")
-  (net 29 "Net-(U1-Pad29)")
-  (net 30 "Net-(U1-Pad28)")
-  (net 31 "Net-(U1-Pad27)")
-  (net 32 "Net-(U1-Pad26)")
-  (net 33 "Net-(U1-Pad25)")
-  (net 34 "Net-(U1-Pad22)")
-  (net 35 "Net-(U1-Pad21)")
-  (net 36 "Net-(U1-Pad20)")
-  (net 37 "Net-(U1-Pad19)")
-  (net 38 "Net-(U1-Pad18)")
-  (net 39 "Net-(U1-Pad12)")
-  (net 40 "Net-(U1-Pad11)")
-  (net 41 "Net-(U1-Pad10)")
-  (net 42 "Net-(U1-Pad9)")
-  (net 43 "Net-(U1-Pad8)")
-  (net 44 "Net-(U1-Pad1)")
-  (net 45 "Net-(USB1-Pad6)")
-  (net 46 "Net-(USB1-Pad2)")
+  (net 26 "Net-(U1-Pad28)")
+  (net 27 "Net-(U1-Pad27)")
+  (net 28 "Net-(U1-Pad26)")
+  (net 29 "Net-(U1-Pad25)")
+  (net 30 "Net-(U1-Pad22)")
+  (net 31 "Net-(U1-Pad21)")
+  (net 32 "Net-(U1-Pad20)")
+  (net 33 "Net-(U1-Pad19)")
+  (net 34 "Net-(U1-Pad18)")
+  (net 35 "Net-(U1-Pad12)")
+  (net 36 "Net-(U1-Pad11)")
+  (net 37 "Net-(U1-Pad10)")
+  (net 38 "Net-(U1-Pad9)")
+  (net 39 "Net-(U1-Pad8)")
+  (net 40 "Net-(U1-Pad1)")
+  (net 41 "Net-(USB1-Pad6)")
+  (net 42 "Net-(USB1-Pad2)")
   (net_class Default "This is the default net class."
     (clearance 0.2)
@@
     (add_net "Net-(U1-Pad27)")
     (add_net "Net-(U1-Pad28)")
-    (add_net "Net-(U1-Pad29)")
-    (add_net "Net-(U1-Pad30)")
-    (add_net "Net-(U1-Pad31)")
-    (add_net "Net-(U1-Pad32)")
     (add_net "Net-(U1-Pad36)")
     (add_net "Net-(U1-Pad37)")
@@
       (net 1 GND))
     (pad 2 smd rect (at 4.5 0.8 270) (size 2.25 0.5) (layers F.Cu F.Paste F.Mask)
-      (net 46 "Net-(USB1-Pad2)"))
+      (net 42 "Net-(USB1-Pad2)"))
     (pad 3 smd rect (at 4.5 0 270) (size 2.25 0.5) (layers F.Cu F.Paste F.Mask)
       (net 15 D+))
@@
       (net 10 VCC))
     (pad 6 thru_hole oval (at 4.5 -3.65 270) (size 2.7 1.7) (drill oval 1.9 0.7) (layers *.Cu *.Mask)
-      (net 45 "Net-(USB1-Pad6)"))
+      (net 41 "Net-(USB1-Pad6)"))
     (pad 6 thru_hole oval (at 4.5 3.65 270) (size 2.7 1.7) (drill oval 1.9 0.7) (layers *.Cu *.Mask)
-      (net 45 "Net-(USB1-Pad6)"))
+      (net 41 "Net-(USB1-Pad6)"))
     (pad 6 thru_hole oval (at 0 3.65 270) (size 2.7 1.7) (drill oval 1.9 0.7) (layers *.Cu *.Mask)
-      (net 45 "Net-(USB1-Pad6)"))
+      (net 41 "Net-(USB1-Pad6)"))
     (pad 6 thru_hole oval (at 0 -3.65 270) (size 2.7 1.7) (drill oval 1.9 0.7) (layers *.Cu *.Mask)
-      (net 45 "Net-(USB1-Pad6)"))
+      (net 41 "Net-(USB1-Pad6)"))
   )
   (module Package_QFP:TQFP-44_10x10mm_P0.8mm (layer F.Cu)
@@
     (fp_line (start -5.175 -4.6) (end -6.45 -4.6) (layer F.SilkS) (width 0.15))
     (pad 1 smd rect (at -5.7 -4) (size 1.5 0.55) (layers F.Cu F.Paste F.Mask)
-      (net 44 "Net-(U1-Pad1)"))
+      (net 40 "Net-(U1-Pad1)"))
     (pad 2 smd rect (at -5.7 -3.2) (size 1.5 0.55) (layers F.Cu F.Paste F.Mask)
       (net 2 +5V))
@@
       (net 2 +5V))
     (pad 8 smd rect (at -5.7 1.6) (size 1.5 0.55) (layers F.Cu F.Paste F.Mask)
-      (net 43 "Net-(U1-Pad8)"))
+      (net 39 "Net-(U1-Pad8)"))
     (pad 9 smd rect (at -5.7 2.4) (size 1.5 0.55) (layers F.Cu F.Paste F.Mask)
-      (net 42 "Net-(U1-Pad9)"))
+      (net 38 "Net-(U1-Pad9)"))
     (pad 10 smd rect (at -5.7 3.2) (size 1.5 0.55) (layers F.Cu F.Paste F.Mask)
-      (net 41 "Net-(U1-Pad10)"))
+      (net 37 "Net-(U1-Pad10)"))
     (pad 11 smd rect (at -5.7 4) (size 1.5 0.55) (layers F.Cu F.Paste F.Mask)
-      (net 40 "Net-(U1-Pad11)"))
+      (net 36 "Net-(U1-Pad11)"))
     (pad 12 smd rect (at -4 5.7 90) (size 1.5 0.55) (layers F.Cu F.Paste F.Mask)
-      (net 39 "Net-(U1-Pad12)"))
+      (net 35 "Net-(U1-Pad12)"))
     (pad 13 smd rect (at -3.2 5.7 90) (size 1.5 0.55) (layers F.Cu F.Paste F.Mask)
       (net 17 "Net-(R3-Pad2)"))
@@
       (net 3 "Net-(C5-Pad1)"))
     (pad 18 smd rect (at 0.8 5.7 90) (size 1.5 0.55) (layers F.Cu F.Paste F.Mask)
-      (net 38 "Net-(U1-Pad18)"))
+      (net 34 "Net-(U1-Pad18)"))
     (pad 19 smd rect (at 1.6 5.7 90) (size 1.5 0.55) (layers F.Cu F.Paste F.Mask)
-      (net 37 "Net-(U1-Pad19)"))
+      (net 33 "Net-(U1-Pad19)"))
     (pad 20 smd rect (at 2.4 5.7 90) (size 1.5 0.55) (layers F.Cu F.Paste F.Mask)
-      (net 36 "Net-(U1-Pad20)"))
+      (net 32 "Net-(U1-Pad20)"))
     (pad 21 smd rect (at 3.2 5.7 90) (size 1.5 0.55) (layers F.Cu F.Paste F.Mask)
-      (net 35 "Net-(U1-Pad21)"))
+      (net 31 "Net-(U1-Pad21)"))
     (pad 22 smd rect (at 4 5.7 90) (size 1.5 0.55) (layers F.Cu F.Paste F.Mask)
-      (net 34 "Net-(U1-Pad22)"))
+      (net 30 "Net-(U1-Pad22)"))
     (pad 23 smd rect (at 5.7 4) (size 1.5 0.55) (layers F.Cu F.Paste F.Mask)
       (net 1 GND))
@@
       (net 2 +5V))
     (pad 25 smd rect (at 5.7 2.4) (size 1.5 0.55) (layers F.Cu F.Paste F.Mask)
-      (net 33 "Net-(U1-Pad25)"))
+      (net 29 "Net-(U1-Pad25)"))
     (pad 26 smd rect (at 5.7 1.6) (size 1.5 0.55) (layers F.Cu F.Paste F.Mask)
-      (net 32 "Net-(U1-Pad26)"))
+      (net 28 "Net-(U1-Pad26)"))
     (pad 27 smd rect (at 5.7 0.8) (size 1.5 0.55) (layers F.Cu F.Paste F.Mask)
-      (net 31 "Net-(U1-Pad27)"))
+      (net 27 "Net-(U1-Pad27)"))
     (pad 28 smd rect (at 5.7 0) (size 1.5 0.55) (layers F.Cu F.Paste F.Mask)
-      (net 30 "Net-(U1-Pad28)"))
+      (net 26 "Net-(U1-Pad28)"))
     (pad 29 smd rect (at 5.7 -0.8) (size 1.5 0.55) (layers F.Cu F.Paste F.Mask)
-      (net 29 "Net-(U1-Pad29)"))
+      (net 11 COL0))
     (pad 30 smd rect (at 5.7 -1.6) (size 1.5 0.55) (layers F.Cu F.Paste F.Mask)
-      (net 28 "Net-(U1-Pad30)"))
+      (net 8 ROW1))
     (pad 31 smd rect (at 5.7 -2.4) (size 1.5 0.55) (layers F.Cu F.Paste F.Mask)
-      (net 27 "Net-(U1-Pad31)"))
+      (net 12 COL1))
     (pad 32 smd rect (at 5.7 -3.2) (size 1.5 0.55) (layers F.Cu F.Paste F.Mask)
-      (net 26 "Net-(U1-Pad32)"))
+      (net 12 COL1))
     (pad 33 smd rect (at 5.7 -4) (size 1.5 0.55) (layers F.Cu F.Paste F.Mask)
       (net 18 "Net-(R4-Pad2)"))
@@
   (segment (start 112.1835 119.325) (end 115.0335 122.175) (width 0.254) (layer F.Cu) (net 7))
   (segment (start 110.45 119.325) (end 112.1835 119.325) (width 0.254) (layer F.Cu) (net 7))
+  (segment (start 153.1335 125.475) (end 153.9875 125.475) (width 0.254) (layer F.Cu) (net 8))
+  (segment (start 152.462599 126.145901) (end 153.1335 125.475) (width 0.254) (layer F.Cu) (net 8))
+  (segment (start 144.935967 126.145901) (end 152.462599 126.145901) (width 0.254) (layer F.Cu) (net 8))
+  (segment (start 144.265066 125.475) (end 144.935967 126.145901) (width 0.254) (layer F.Cu) (net 8))
+  (segment (start 134.9375 125.475) (end 144.265066 125.475) (width 0.254) (layer F.Cu) (net 8))
+  (segment (start 134.9375 126.179) (end 134.9375 125.475) (width 0.254) (layer F.Cu) (net 8))
+  (segment (start 136.41852 127.66002) (end 134.9375 126.179) (width 0.254) (layer F.Cu) (net 8))
+  (segment (start 136.41852 140.94173) (end 136.41852 127.66002) (width 0.254) (layer F.Cu) (net 8))
+  (segment (start 133.704 143.65625) (end 136.41852 140.94173) (width 0.254) (layer F.Cu) (net 8))
+  (segment (start 132.7 143.65625) (end 133.704 143.65625) (width 0.254) (layer F.Cu) (net 8))
   (segment (start 130.12 119.325) (end 129.5 119.325) (width 0.254) (layer F.Cu) (net 9))
   (segment (start 132.97 122.175) (end 130.12 119.325) (width 0.254) (layer F.Cu) (net 9))
@@
   (segment (start 124.5 119.825) (end 124.5 103.545) (width 0.254) (layer B.Cu) (net 11))
   (via (at 123.19 102.235) (size 0.8) (drill 0.4) (layers F.Cu B.Cu) (net 11))
+  (via (at 134.14375 144.4625) (size 0.8) (drill 0.4) (layers F.Cu B.Cu) (net 11))
+  (segment (start 132.7 144.45625) (end 134.1375 144.45625) (width 0.254) (layer F.Cu) (net 11))
+  (segment (start 134.1375 144.45625) (end 134.14375 144.4625) (width 0.254) (layer F.Cu) (net 11))
+  (segment (start 126.09099 119.825) (end 124.5 119.825) (width 0.254) (layer B.Cu) (net 11))
+  (segment (start 126.301038 119.825) (end 126.09099 119.825) (width 0.254) (layer B.Cu) (net 11))
+  (segment (start 134.14375 127.667712) (end 126.301038 119.825) (width 0.254) (layer B.Cu) (net 11))
+  (segment (start 134.14375 144.4625) (end 134.14375 127.667712) (width 0.254) (layer B.Cu) (net 11))
   (segment (start 115.8875 124.771) (end 115.8875 125.475) (width 0.254) (layer F.Cu) (net 12))
   (segment (start 112.4015 121.285) (end 115.8875 124.771) (width 0.254) (layer F.Cu) (net 12))
@@
   (segment (start 134.9375 111.2125) (end 143.55 119.825) (width 0.254) (layer F.Cu) (net 12))
   (segment (start 134.9375 106.425) (end 134.9375 111.2125) (width 0.254) (layer F.Cu) (net 12))
+  (segment (start 132.7 142.05625) (end 132.7 142.85625) (width 0.254) (layer F.Cu) (net 12))
+  (segment (start 116.7415 125.475) (end 115.8875 125.475) (width 0.254) (layer F.Cu) (net 12))
+  (segment (start 123.950928 125.475) (end 116.7415 125.475) (width 0.254) (layer F.Cu) (net 12))
+  (segment (start 135.96451 137.488582) (end 123.950928 125.475) (width 0.254) (layer F.Cu) (net 12))
+  (segment (start 135.96451 140.323918) (end 135.96451 137.488582) (width 0.254) (layer F.Cu) (net 12))
+  (segment (start 134.232178 142.05625) (end 135.96451 140.323918) (width 0.254) (layer F.Cu) (net 12))
+  (segment (start 132.7 142.05625) (end 134.232178 142.05625) (width 0.254) (layer F.Cu) (net 12))
   (via (at 109.743753 104.775) (size 0.8) (drill 0.4) (layers F.Cu B.Cu) (net 13))
   (segment (start 109.54375 101.3375) (end 109.54375 104.574997) (width 0.254) (layer F.Cu) (net 13))
