File: first-3k-keypad.kicad_pcb (KiCad board)
At the start: 2 copper layers, 57.1 x 71.4 mm, 24 parts, among them SW1 SW_Push, U1 ATmega32U4-AU, Y1 16MHz

Commit message: New Trace Layout
Parts:
- moved C3 21.1 mm to (114.3, 149.2), turned to 90 degrees
- moved F1 18.0 mm to (131.0, 135.7), turned to 180 degrees
- moved C4 13.9 mm to (139.7, 144.5), turned to 270 degrees
- moved C1 12.7 mm to (111.1, 136.5), turned to 90 degrees
- moved R3 5.94 mm to (114.3, 155.6), turned to 270 degrees
- moved R1 5.84 mm to (122.2, 135.7), turned to 180 degrees
- moved C7 5.02 mm to (114.3, 142.9)
- moved C2 5.02 mm to (139.7, 150.8)
- moved R4 4.83 mm to (139.7, 138.1), turned to 90 degrees
- moved R2 3.27 mm to (116.7, 136.5), turned to 90 degrees
- moved C5 2.86 mm to (121.4, 155.6)
- moved C6 2.86 mm to (132.6, 155.6)
- moved SW1 2.38 mm to (127.0, 161.9), turned to 0 degrees
- moved Y1 1.59 mm to (127.0, 155.6)
Connections:
- U1 pad 27: Net-(U1-Pad27) -> COL1
- U1 pad 28: Net-(U1-Pad28) -> ROW1
- U1 pad 30: ROW1 -> COL1
- U1 pad 31: COL1 -> Net-(U1-Pad31)
- U1 pad 32: COL1 -> Net-(U1-Pad32)
Routing:
- net +5V: track 50.6 -> 73.7 mm, vias 9 -> 2
- net GND: track 120.0 -> 134.9 mm, vias 2 -> 8
- net VCC: track 50.6 -> 42.4 mm
- net D+: track 45.7 -> 37.5 mm
- net Net-(C7-Pad1): track 0.00 -> 7.60 mm, vias 0 -> 3
- net Net-(R4-Pad2): track 2.82 -> 9.00 mm
- net Net-(R1-Pad1): track 3.03 -> 8.51 mm, vias 0 -> 2
- net COL1: track 102.5 -> 107.7 mm, vias 0 -> 2
- net Net-(C5-Pad1): track 7.01 -> 11.0 mm
- net Net-(C6-Pad1): track 12.8 -> 9.11 mm, vias 0 -> 2
- net D-: track 42.3 -> 39.3 mm
- net ROW1: track 40.5 -> 41.7 mm, vias 0 -> 3
- net COL0: track 49.3 -> 48.2 mm
- net Net-(R3-Pad2): track 21.2 -> 20.2 mm
- net Net-(R2-Pad1): track 9.38 -> 8.97 mm, vias 0 -> 2

Commit message: Gounds, deco
Routing:
- added copper zone on F.Cu, net GND
Other:
- board text added: "The phrase “it’s just a game” is such a weak mindset. You are ok with what happened, losing, imperfection of a craft. When you stop getting angry after losing, you’ve lost twice. There’s always something to learn, and always room for improvement, never settle."
Changed lines of the file:
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@@
   (general
     (thickness 1.6)
-    (drawings 9)
+    (drawings 10)
     (tracks 203)
     (zones 0)
@@
     (visible_elements 7FFFFFFF)
     (pcbplotparams
-      (layerselection 0x010fc_ffffffff)
-      (usegerberextensions false)
+      (layerselection 0x010f0_ffffffff)
+      (usegerberextensions true)
       (usegerberattributes false)
       (usegerberadvancedattributes false)
       (creategerberjobfile false)
       (excludeedgelayer true)
-      (linewidth 0.100000)
+      (linewidth 0.020000)
       (plotframeref false)
       (viasonmask false)
@@
       (plotinvisibletext false)
       (padsonsilk false)
-      (subtractmaskfromsilk false)
+      (subtractmaskfromsilk true)
       (outputformat 1)
       (mirror false)
-      (drillshape 1)
+      (drillshape 0)
       (scaleselection 1)
       (outputdirectory ""))
@@
       (rotate (xyz 0 0 0))
     )
+  )
+  (gr_text "The phrase “it’s just a game” is such a weak mindset. \nYou are ok with what happened, losing, imperfection \nof a craft. When you stop getting angry after losing, \nyou’ve lost twice. There’s always something to learn, \nand always room for improvement, never settle." (at 127 112.7125) (layer B.SilkS)
+    (effects (font (size 1 1) (thickness 0.15)) (justify mirror))
   )
   (gr_line (start 151.60625 95.25) (end 150.8125 95.25) (layer Edge.Cuts) (width 0.05))
@@
   (segment (start 136.25225 137.175) (end 132.7 140.72725) (width 0.254) (layer F.Cu) (net 18))
   (segment (start 139.7 137.175) (end 136.25225 137.175) (width 0.254) (layer F.Cu) (net 18))
+  (zone (net 1) (net_name GND) (layer F.Cu) (hatch edge 0.508)
+    (connect_pads (clearance 0.508))
+    (min_thickness 0.254)
+    (fill yes (arc_segments 32) (thermal_gap 0.508) (thermal_bridge_width 0.508))
+    (polygon
+      (pts
+        (xy 109.5375 134.14375) (xy 109.5375 138.90625) (xy 112.7125 142.08125) (xy 112.7125 157.95625) (xy 117.475 162.71875)
+        (xy 119.85625 165.1) (xy 131.7625 165.1) (xy 141.2875 157.1625) (xy 141.2875 135.73125) (xy 139.7 134.14375)
+      )
+    )
+  )
+  (zone (net 1) (net_name GND) (layer F.Cu) (hatch edge 0.508)
+    (connect_pads (clearance 0.508))
+    (min_thickness 0.254)
+    (fill yes (arc_segments 32) (thermal_gap 0.508) (thermal_bridge_width 0.508))
+    (polygon
+      (pts
+        (xy 103.1875 95.25) (xy 103.1875 102.39375) (xy 104.775 103.98125) (xy 111.91875 103.98125) (xy 112.7125 103.98125)
+        (xy 114.3 102.39375) (xy 114.3 95.25)
+      )
+    )
+  )
 )

Commit message: Updated Traces
Parts:
- moved R1 31.0 mm to (110.3, 107.2), turned to 90 degrees
- moved R2 30.6 mm to (108.0, 107.2)
- moved C1 27.0 mm to (134.9, 149.2), turned to 270 degrees
- moved C4 17.4 mm to (123.8, 137.3), turned to 0 degrees
- moved C2 16.1 mm to (131.0, 137.3), turned to 180 degrees
- moved F1 10.3 mm to (120.7, 135.7), turned to 90 degrees
- moved R3 7.32 mm to (119.1, 150.0)
- moved C3 6.20 mm to (119.1, 145.3)
- moved R4 5.02 mm to (134.9, 139.7), turned to 270 degrees
- moved C7 2.86 mm to (116.7, 144.5)
- moved USB1 0.79 mm to (108.7, 97.6)
Routing:
- net D-: track 39.3 -> 4.41 mm, vias 2 -> 0
- net D+: track 37.5 -> 4.42 mm, vias 2 -> 0
- net Net-(R2-Pad1): track 8.97 -> 41.9 mm, vias 2 -> 0
- net Net-(R1-Pad1): track 8.51 -> 40.4 mm, vias 2 -> 0
- net GND: track 134.9 -> 108.0 mm, vias 8 -> 0
- net COL1: track 107.7 -> 123.5 mm, vias 2 -> 3
- net COL0: track 48.2 -> 57.3 mm, vias 3 -> 0
- net Net-(R4-Pad2): track 9.00 -> 2.80 mm
- net +5V: track 73.7 -> 68.2 mm, vias 2 -> 5
- net VCC: track 42.4 -> 37.3 mm, vias 2 -> 0
- net Net-(C7-Pad1): track 7.60 -> 4.68 mm, vias 3 -> 0
- net Net-(R3-Pad2): track 20.2 -> 18.6 mm, vias 2 -> 0
- net ROW1: track 41.7 -> 42.8 mm, vias 3 -> 0
- net Net-(C5-Pad1): track 11.0 -> 11.3 mm, vias 0 -> 2
- net Net-(C6-Pad1): vias 2 -> 0
