File: first-3k-keypad.kicad_pcb (KiCad board)
At the start: 2 copper layers, 57.1 x 71.4 mm, 24 parts, among them SW1 SW_Push, U1 ATmega32U4-AU, Y1 16MHz

Commit message: 3552662432235523235
Parts:
- moved USB1 0.79 mm to (108.7, 96.8)
Routing:
- net VCC: track 38.2 -> 39.0 mm
- net GND: track 109.4 -> 110.2 mm
- net D-: track 4.41 -> 5.21 mm
- net D+: track 4.42 -> 5.21 mm
Changed lines of the file:
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@@
   )
   (module random-keyboard-parts:Molex-0548190589 (layer F.Cu)
-    (at 108.74375 97.63125 270)
+    (at 108.74375 96.8375 270)
     (attr smd)
     (fp_text reference USB1 (at 2.032 0) (layer F.SilkS)
@@
   (segment (start 118.26875 132.55625) (end 117.475 133.35) (width 0.381) (layer F.Cu) (net 1))
   (segment (start 118.26875 121.44375) (end 118.26875 132.55625) (width 0.381) (layer F.Cu) (net 1))
-  (segment (start 107.14375 103.00625) (end 107.15625 103.01875) (width 0.381) (layer F.Cu) (net 1))
-  (segment (start 107.14375 102.13125) (end 107.14375 103.00625) (width 0.381) (layer F.Cu) (net 1))
-  (segment (start 107.15625 103.01875) (end 107.15625 103.98125) (width 0.381) (layer F.Cu) (net 1))
+  (segment (start 107.14375 101.3375) (end 107.14375 102.2125) (width 0.381) (layer F.Cu) (net 1))
+  (segment (start 107.15625 102.225) (end 107.15625 103.98125) (width 0.381) (layer F.Cu) (net 1))
   (segment (start 107.15625 103.98125) (end 105.56875 105.56875) (width 0.381) (layer F.Cu) (net 1))
+  (segment (start 105.56875 108.74375) (end 118.26875 121.44375) (width 0.381) (layer F.Cu) (net 1))
+  (segment (start 107.14375 102.2125) (end 107.15625 102.225) (width 0.381) (layer F.Cu) (net 1))
   (segment (start 105.56875 105.56875) (end 105.56875 108.74375) (width 0.381) (layer F.Cu) (net 1))
-  (segment (start 105.56875 108.74375) (end 118.26875 121.44375) (width 0.381) (layer F.Cu) (net 1))
   (segment (start 119.2 146.05625) (end 121.3 146.05625) (width 0.381) (layer F.Cu) (net 2))
   (segment (start 119.0625 146.19375) (end 119.2 146.05625) (width 0.381) (layer F.Cu) (net 2))
@@
   (segment (start 120.65 133.24075) (end 120.65 134.33125) (width 0.381) (layer F.Cu) (net 10))
   (segment (start 110.34375 104.63427) (end 111.77802 104.63427) (width 0.381) (layer F.Cu) (net 10))
-  (segment (start 110.34375 102.13125) (end 110.34375 104.63427) (width 0.381) (layer F.Cu) (net 10))
   (segment (start 111.77802 104.63427) (end 111.77802 112.57177) (width 0.381) (layer F.Cu) (net 10))
   (segment (start 111.77802 112.57177) (end 119.9655 120.75925) (width 0.381) (layer F.Cu) (net 10))
   (segment (start 119.9655 120.75925) (end 119.9655 132.55625) (width 0.381) (layer F.Cu) (net 10))
   (segment (start 119.9655 132.55625) (end 120.65 133.24075) (width 0.381) (layer F.Cu) (net 10))
+  (segment (start 110.34375 101.3375) (end 110.34375 104.63427) (width 0.381) (layer F.Cu) (net 10))
   (segment (start 123.19 118.515) (end 123.19 121.285) (width 0.254) (layer F.Cu) (net 11))
   (segment (start 123.19 102.235) (end 123.19 118.515) (width 0.254) (layer F.Cu) (net 11))
@@
   (segment (start 104.14 121.135) (end 104.14 121.285) (width 0.254) (layer B.Cu) (net 12))
   (segment (start 109.54375 105.43125) (end 110.33125 106.21875) (width 0.254) (layer F.Cu) (net 13))
-  (segment (start 109.54375 102.13125) (end 109.54375 105.43125) (width 0.254) (layer F.Cu) (net 13))
+  (segment (start 109.54375 105.43125) (end 109.54375 101.3375) (width 0.254) (layer F.Cu) (net 13))
   (segment (start 121.1375 143.01875) (end 121.3 142.85625) (width 0.254) (layer F.Cu) (net 14))
   (segment (start 120.296 142.85625) (end 121.3 142.85625) (width 0.254) (layer F.Cu) (net 14))
@@
   (segment (start 118.446521 133.752413) (end 118.446521 141.465271) (width 0.254) (layer F.Cu) (net 14))
   (segment (start 108.74375 105.425) (end 107.95 106.21875) (width 0.254) (layer F.Cu) (net 15))
-  (segment (start 108.74375 102.13125) (end 108.74375 105.425) (width 0.254) (layer F.Cu) (net 15))
+  (segment (start 108.74375 101.3375) (end 108.74375 105.425) (width 0.254) (layer F.Cu) (net 15))
   (segment (start 107.95 108.09375) (end 107.95 108.74375) (width 0.254) (layer F.Cu) (net 16))
   (segment (start 119.907178 143.65625) (end 120.296 143.65625) (width 0.254) (layer F.Cu) (net 16))
@@
     (polygon
       (pts
-        (xy 114.3 95.25) (xy 114.3 110.33125) (xy 103.1875 110.33125) (xy 103.1875 95.25)
+        (xy 114.3 95.25) (xy 114.3 110.352142) (xy 103.1875 110.352142) (xy 103.1875 95.25)
       )
     )
