File: first-3k-keypad.sch (KiCad schematic (older format))
At the start: 1 part

Commit message: 4
Parts:
- added C?: 1uF, symbol Device:C_Small
- added R?: 10k, symbol Device:R_Small
- added R? (x2): 22, symbol Device:R_Small
Connections:
- wire segments 5 -> 13
Changed lines of the file:
@@
 	5700 5700 5350 5700
 Connection ~ 5700 5700
+$Comp
+L Device:R_Small R?
+U 1 1 634120A0
+P 7150 4500
+F 0 "R?" V 6954 4500 50  0000 C CNN
+F 1 "10k" V 7045 4500 50  0000 C CNN
+F 2 "" H 7150 4500 50  0001 C CNN
+F 3 "~" H 7150 4500 50  0001 C CNN
+	1    7150 4500
+	0    1    1    0
+$EndComp
+$Comp
+L power:GND #PWR?
+U 1 1 63418816
+P 7600 4500
+F 0 "#PWR?" H 7600 4250 50  0001 C CNN
+F 1 "GND" H 7605 4327 50  0000 C CNN
+F 2 "" H 7600 4500 50  0001 C CNN
+F 3 "" H 7600 4500 50  0001 C CNN
+	1    7600 4500
+	1    0    0    -1
+$EndComp
+Wire Wire Line
+	6400 4500 7050 4500
+Wire Wire Line
+	7250 4500 7600 4500
+$Comp
+L Device:R_Small R?
+U 1 1 6341A326
+P 4600 3400
+F 0 "R?" V 4404 3400 50  0000 C CNN
+F 1 "22" V 4495 3400 50  0000 C CNN
+F 2 "" H 4600 3400 50  0001 C CNN
+F 3 "~" H 4600 3400 50  0001 C CNN
+	1    4600 3400
+	0    1    1    0
+$EndComp
+$Comp
+L Device:R_Small R?
+U 1 1 6341B15B
+P 4200 3500
+F 0 "R?" V 4004 3500 50  0000 C CNN
+F 1 "22" V 4095 3500 50  0000 C CNN
+F 2 "" H 4200 3500 50  0001 C CNN
+F 3 "~" H 4200 3500 50  0001 C CNN
+	1    4200 3500
+	0    1    1    0
+$EndComp
+Wire Wire Line
+	5200 3400 4700 3400
+Wire Wire Line
+	5200 3500 4300 3500
+Wire Wire Line
+	4500 3400 4000 3400
+Wire Wire Line
+	4100 3500 4000 3500
+$Comp
+L Device:C_Small C?
+U 1 1 6341E127
+P 4750 3800
+F 0 "C?" H 4842 3846 50  0000 L CNN
+F 1 "1uF" H 4842 3755 50  0000 L CNN
+F 2 "" H 4750 3800 50  0001 C CNN
+F 3 "~" H 4750 3800 50  0001 C CNN
+	1    4750 3800
+	1    0    0    -1
+$EndComp
+Wire Wire Line
+	5200 3700 4750 3700
+$Comp
+L power:GND #PWR?
+U 1 1 634208DE
+P 4750 4050
+F 0 "#PWR?" H 4750 3800 50  0001 C CNN
+F 1 "GND" H 4755 3877 50  0000 C CNN
+F 2 "" H 4750 4050 50  0001 C CNN
+F 3 "" H 4750 4050 50  0001 C CNN
+	1    4750 4050
+	1    0    0    -1
+$EndComp
+Wire Wire Line
+	4750 3900 4750 4050
 $EndSCHEMATC

Commit message: 5
Parts:
- added C? (x3): 0.1uf, symbol Device:C_Small
- added C?: 10uf, symbol Device:C_Small
- added Y?: 16MHz, symbol Device:Crystal_GND24_Small
Connections:
- wire segments 13 -> 24
Changed lines of the file:
@@
 EESchema Schematic File Version 4
+LIBS:first-3k-keypad-cache
 EELAYER 30 0
 EELAYER END
@@
 Wire Wire Line
 	4750 3900 4750 4050
+$Comp
+L Device:C_Small C?
+U 1 1 6351BB14
+P 3000 4150
+F 0 "C?" H 3092 4196 50  0000 L CNN
+F 1 "0.1uf" H 3092 4105 50  0000 L CNN
+F 2 "" H 3000 4150 50  0001 C CNN
+F 3 "~" H 3000 4150 50  0001 C CNN
+	1    3000 4150
+	1    0    0    -1
+$EndComp
+$Comp
+L Device:C_Small C?
+U 1 1 6351E0C3
+P 3350 4150
+F 0 "C?" H 3442 4196 50  0000 L CNN
+F 1 "0.1uf" H 3442 4105 50  0000 L CNN
+F 2 "" H 3350 4150 50  0001 C CNN
+F 3 "~" H 3350 4150 50  0001 C CNN
+	1    3350 4150
+	1    0    0    -1
+$EndComp
+$Comp
+L Device:C_Small C?
+U 1 1 6351EB38
+P 3750 4150
+F 0 "C?" H 3842 4196 50  0000 L CNN
+F 1 "0.1uf" H 3842 4105 50  0000 L CNN
+F 2 "" H 3750 4150 50  0001 C CNN
+F 3 "~" H 3750 4150 50  0001 C CNN
+	1    3750 4150
+	1    0    0    -1
+$EndComp
+$Comp
+L Device:C_Small C?
+U 1 1 6351EE1A
+P 4150 4150
+F 0 "C?" H 4242 4196 50  0000 L CNN
+F 1 "10uf" H 4242 4105 50  0000 L CNN
+F 2 "" H 4150 4150 50  0001 C CNN
+F 3 "~" H 4150 4150 50  0001 C CNN
+	1    4150 4150
+	1    0    0    -1
+$EndComp
+Wire Wire Line
+	3000 4050 3350 4050
+Connection ~ 3350 4050
+Connection ~ 3750 4050
+Wire Wire Line
+	3750 4050 4150 4050
+Wire Wire Line
+	3000 4250 3350 4250
+Connection ~ 3350 4250
+Connection ~ 3750 4250
+Wire Wire Line
+	3750 4250 4150 4250
+Wire Wire Line
+	3350 4050 3550 4050
+Wire Wire Line
+	3350 4250 3550 4250
+Wire Wire Line
+	3550 4050 3550 4000
+Connection ~ 3550 4050
+Wire Wire Line
+	3550 4050 3750 4050
+Wire Wire Line
+	3550 4250 3550 4300
+Connection ~ 3550 4250
+Wire Wire Line
+	3550 4250 3750 4250
+$Comp
+L power:GND #PWR?
+U 1 1 63524E27
+P 3550 4300
+F 0 "#PWR?" H 3550 4050 50  0001 C CNN
+F 1 "GND" H 3555 4127 50  0000 C CNN
+F 2 "" H 3550 4300 50  0001 C CNN
+F 3 "" H 3550 4300 50  0001 C CNN
+	1    3550 4300
+	1    0    0    -1
+$EndComp
+$Comp
+L power:+5V #PWR?
+U 1 1 63525888
+P 3550 4000
+F 0 "#PWR?" H 3550 3850 50  0001 C CNN
+F 1 "+5V" H 3565 4173 50  0000 C CNN
+F 2 "" H 3550 4000 50  0001 C CNN
+F 3 "" H 3550 4000 50  0001 C CNN
+	1    3550 4000
+	1    0    0    -1
+$EndComp
+Wire Wire Line
+	5200 3200 4750 3200
+$Comp
+L power:+5V #PWR?
+U 1 1 63526C97
+P 4750 3200
+F 0 "#PWR?" H 4750 3050 50  0001 C CNN
+F 1 "+5V" H 4765 3373 50  0000 C CNN
+F 2 "" H 4750 3200 50  0001 C CNN
+F 3 "" H 4750 3200 50  0001 C CNN
+	1    4750 3200
+	1    0    0    -1
+$EndComp
+$Comp
+L Device:Crystal_GND24_Small Y?
+U 1 1 6352765E
+P 4550 2700
+F 0 "Y?" H 4694 2746 50  0000 L CNN
+F 1 "16MHz" H 4694 2655 50  0000 L CNN
+F 2 "" H 4550 2700 50  0001 C CNN
+F 3 "~" H 4550 2700 50  0001 C CNN
+	1    4550 2700
+	1    0    0    -1
+$EndComp
 $EndSCHEMATC

Commit message: 6
Parts:
- added C? (x2): 22pF, symbol Device:C_Small
- added R?: 10k, symbol Device:R_Small
- added SW?: SW_Push, symbol Switch:SW_Push
Connections:
- net labels added: D+, D-
- wire segments 24 -> 41
Changed lines of the file:
@@
 U 1 1 6352765E
 P 4550 2700
-F 0 "Y?" H 4694 2746 50  0000 L CNN
-F 1 "16MHz" H 4694 2655 50  0000 L CNN
+F 0 "Y?" V 4504 2844 50  0000 L CNN
+F 1 "16MHz" V 4595 2844 50  0000 L CNN
 F 2 "" H 4550 2700 50  0001 C CNN
 F 3 "~" H 4550 2700 50  0001 C CNN
 	1    4550 2700
+	0    1    1    0
+$EndComp
+Wire Wire Line
+	5200 2600 4550 2600
+Wire Wire Line
+	4550 2800 5200 2800
+$Comp
+L power:GND #PWR?
+U 1 1 6352B32F
+P 4100 2900
+F 0 "#PWR?" H 4100 2650 50  0001 C CNN
+F 1 "GND" H 4105 2727 50  0000 C CNN
+F 2 "" H 4100 2900 50  0001 C CNN
+F 3 "" H 4100 2900 50  0001 C CNN
+	1    4100 2900
 	1    0    0    -1
 $EndComp
+$Comp
+L Device:C_Small C?
+U 1 1 6352BF05
+P 4200 2550
+F 0 "C?" V 3971 2550 50  0000 C CNN
+F 1 "22pF" V 4062 2550 50  0000 C CNN
+F 2 "" H 4200 2550 50  0001 C CNN
+F 3 "~" H 4200 2550 50  0001 C CNN
+	1    4200 2550
+	0    1    1    0
+$EndComp
+$Comp
+L Device:C_Small C?
+U 1 1 6352CD4F
+P 4200 2850
+F 0 "C?" V 3971 2850 50  0000 C CNN
+F 1 "22pF" V 4062 2850 50  0000 C CNN
+F 2 "" H 4200 2850 50  0001 C CNN
+F 3 "~" H 4200 2850 50  0001 C CNN
+	1    4200 2850
+	0    1    1    0
+$EndComp
+Wire Wire Line
+	4300 2550 4550 2550
+Wire Wire Line
+	4550 2550 4550 2600
+Connection ~ 4550 2600
+Wire Wire Line
+	4550 2800 4550 2850
+Wire Wire Line
+	4550 2850 4300 2850
+Connection ~ 4550 2800
+Wire Wire Line
+	4100 2550 4100 2850
+Connection ~ 4100 2850
+Wire Wire Line
+	4100 2850 4100 2900
+Wire Wire Line
+	4100 2900 4450 2900
+Wire Wire Line
+	4450 2900 4450 2700
+Connection ~ 4100 2900
+Wire Wire Line
+	4450 2900 4650 2900
+Wire Wire Line
+	4650 2900 4650 2700
+Connection ~ 4450 2900
+$Comp
+L Switch:SW_Push SW?
+U 1 1 6353358D
+P 4900 2400
+F 0 "SW?" H 4900 2685 50  0000 C CNN
+F 1 "SW_Push" H 4900 2594 50  0000 C CNN
+F 2 "" H 4900 2600 50  0001 C CNN
+F 3 "~" H 4900 2600 50  0001 C CNN
+	1    4900 2400
+	1    0    0    -1
+$EndComp
+$Comp
+L power:GND #PWR?
+U 1 1 6353478A
+P 4600 2400
+F 0 "#PWR?" H 4600 2150 50  0001 C CNN
+F 1 "GND" H 4605 2227 50  0000 C CNN
+F 2 "" H 4600 2400 50  0001 C CNN
+F 3 "" H 4600 2400 50  0001 C CNN
+	1    4600 2400
+	1    0    0    -1
+$EndComp
+Wire Wire Line
+	4600 2400 4700 2400
+Wire Wire Line
+	5100 2400 5150 2400
+Wire Wire Line
+	5150 2400 5150 2150
+Connection ~ 5150 2400
+Wire Wire Line
+	5150 2400 5200 2400
+$Comp
+L Device:R_Small R?
+U 1 1 635389FC
+P 5150 2050
+F 0 "R?" H 5209 2096 50  0000 L CNN
+F 1 "10k" H 5209 2005 50  0000 L CNN
+F 2 "" H 5150 2050 50  0001 C CNN
+F 3 "~" H 5150 2050 50  0001 C CNN
+	1    5150 2050
+	1    0    0    -1
+$EndComp
+$Comp
+L power:+5V #PWR?
+U 1 1 6353B908
+P 5150 1850
+F 0 "#PWR?" H 5150 1700 50  0001 C CNN
+F 1 "+5V" H 5165 2023 50  0000 C CNN
+F 2 "" H 5150 1850 50  0001 C CNN
+F 3 "" H 5150 1850 50  0001 C CNN
+	1    5150 1850
+	1    0    0    -1
+$EndComp
+Wire Wire Line
+	5150 1850 5150 1950
+Text GLabel 4000 3400 0    50   Input ~ 0
+D+
+Text GLabel 4000 3500 0    50   Input ~ 0
+D-
 $EndSCHEMATC

Commit message: Finished Schematic
Parts:
- added D? (x4): D_Small, symbol Device:D_Small
- added F?: 500mA, symbol Device:Polyfuse_Small
- added MX? (x4): MX-NoLED, symbol MX_Alps_Hybrid:MX-NoLED
- added USB?: Molex-0548190589, symbol random-keyboard-parts:Molex-0548190589
Connections:
- net +5V: now also F?.1
- net D+: now also USB?.3 (D+)
- net D-: now also USB?.4 (D-)
- net GND: now also USB?.1 (GND)
- new net: D?.2 (A), MX?.2 (ROW) (x4)
- new net COL0: MX?.1 (COL), MX?.1 (COL)
- new net COL1: MX?.1 (COL), MX?.1 (COL)
- new net ROW0: D?.1 (K), D?.1 (K)
- new net ROW1: D?.1 (K), D?.1 (K)
- new net VCC: F?.2, USB?.5 (VBUS)
Changed lines of the file:
@@
 Text GLabel 4000 3500 0    50   Input ~ 0
 D-
+$Comp
+L random-keyboard-parts:Molex-0548190589 USB?
+U 1 1 6353D7B6
+P 7900 1700
+F 0 "USB?" V 8437 1667 60  0000 C CNN
+F 1 "Molex-0548190589" V 8331 1667 60  0000 C CNN
+F 2 "" H 7900 1700 60  0001 C CNN
+F 3 "" H 7900 1700 60  0001 C CNN
+	1    7900 1700
+	0    -1   -1   0
+$EndComp
+$Comp
+L Device:Polyfuse_Small F?
+U 1 1 6353F2F1
+P 9250 1500
+F 0 "F?" V 9045 1500 50  0000 C CNN
+F 1 "500mA" V 9136 1500 50  0000 C CNN
+F 2 "" H 9300 1300 50  0001 L CNN
+F 3 "~" H 9250 1500 50  0001 C CNN
+	1    9250 1500
+	0    1    1    0
+$EndComp
+$Comp
+L power:+5V #PWR?
+U 1 1 63542566
+P 9800 1500
+F 0 "#PWR?" H 9800 1350 50  0001 C CNN
+F 1 "+5V" H 9815 1673 50  0000 C CNN
+F 2 "" H 9800 1500 50  0001 C CNN
+F 3 "" H 9800 1500 50  0001 C CNN
+	1    9800 1500
+	1    0    0    -1
+$EndComp
+Wire Wire Line
+	9800 1500 9350 1500
+$Comp
+L power:VCC #PWR?
+U 1 1 63543A2B
+P 8700 1500
+F 0 "#PWR?" H 8700 1350 50  0001 C CNN
+F 1 "VCC" H 8717 1673 50  0000 C CNN
+F 2 "" H 8700 1500 50  0001 C CNN
+F 3 "" H 8700 1500 50  0001 C CNN
+	1    8700 1500
+	1    0    0    -1
+$EndComp
+Wire Wire Line
+	8200 1500 8700 1500
+Connection ~ 8700 1500
+Wire Wire Line
+	8700 1500 9150 1500
+Text GLabel 8200 1600 2    50   Input ~ 0
+D-
+Text GLabel 8200 1700 2    50   Input ~ 0
+D+
+$Comp
+L power:GND #PWR?
+U 1 1 63546D0F
+P 8300 1900
+F 0 "#PWR?" H 8300 1650 50  0001 C CNN
+F 1 "GND" H 8305 1727 50  0000 C CNN
+F 2 "" H 8300 1900 50  0001 C CNN
+F 3 "" H 8300 1900 50  0001 C CNN
+	1    8300 1900
+	1    0    0    -1
+$EndComp
+Wire Wire Line
+	8300 1900 8200 1900
+$Comp
+L MX_Alps_Hybrid:MX-NoLED MX?
+U 1 1 63548E84
+P 9950 3500
+F 0 "MX?" H 9983 3723 60  0000 C CNN
+F 1 "MX-NoLED" H 9983 3649 20  0000 C CNN
+F 2 "" H 9325 3475 60  0001 C CNN
+F 3 "" H 9325 3475 60  0001 C CNN
+	1    9950 3500
+	1    0    0    -1
+$EndComp
+$Comp
+L Device:D_Small D?
+U 1 1 6354A380
+P 9700 3750
+F 0 "D?" V 9746 3682 50  0000 R CNN
+F 1 "D_Small" V 9655 3682 50  0000 R CNN
+F 2 "" V 9700 3750 50  0001 C CNN
+F 3 "~" V 9700 3750 50  0001 C CNN
+	1    9700 3750
+	0    -1   -1   0
+$EndComp
+Wire Wire Line
+	9700 3650 9900 3650
+$Comp
+L MX_Alps_Hybrid:MX-NoLED MX?
+U 1 1 63552C0D
+P 10600 3500
+F 0 "MX?" H 10633 3723 60  0000 C CNN
+F 1 "MX-NoLED" H 10633 3649 20  0000 C CNN
+F 2 "" H 9975 3475 60  0001 C CNN
+F 3 "" H 9975 3475 60  0001 C CNN
+	1    10600 3500
+	1    0    0    -1
+$EndComp
+$Comp
+L Device:D_Small D?
+U 1 1 63552C17
+P 10350 3750
+F 0 "D?" V 10396 3682 50  0000 R CNN
+F 1 "D_Small" V 10305 3682 50  0000 R CNN
+F 2 "" V 10350 3750 50  0001 C CNN
+F 3 "~" V 10350 3750 50  0001 C CNN
+	1    10350 3750
+	0    -1   -1   0
+$EndComp
+Wire Wire Line
+	10350 3650 10550 3650
+$Comp
+L MX_Alps_Hybrid:MX-NoLED MX?
+U 1 1 63556D1C
+P 9950 4150
+F 0 "MX?" H 9983 4373 60  0000 C CNN
+F 1 "MX-NoLED" H 9983 4299 20  0000 C CNN
+F 2 "" H 9325 4125 60  0001 C CNN
+F 3 "" H 9325 4125 60  0001 C CNN
+	1    9950 4150
+	1    0    0    -1
+$EndComp
+$Comp
+L Device:D_Small D?
+U 1 1 63556D26
+P 9700 4400
+F 0 "D?" V 9746 4332 50  0000 R CNN
+F 1 "D_Small" V 9655 4332 50  0000 R CNN
+F 2 "" V 9700 4400 50  0001 C CNN
+F 3 "~" V 9700 4400 50  0001 C CNN
+	1    9700 4400
+	0    -1   -1   0
+$EndComp
+Wire Wire Line
+	9700 4300 9900 4300
+$Comp
+L MX_Alps_Hybrid:MX-NoLED MX?
+U 1 1 63559CA6
+P 10600 4150
+F 0 "MX?" H 10633 4373 60  0000 C CNN
+F 1 "MX-NoLED" H 10633 4299 20  0000 C CNN
+F 2 "" H 9975 4125 60  0001 C CNN
+F 3 "" H 9975 4125 60  0001 C CNN
+	1    10600 4150
+	1    0    0    -1
+$EndComp
+$Comp
+L Device:D_Small D?
+U 1 1 63559CB0
+P 10350 4400
+F 0 "D?" V 10396 4332 50  0000 R CNN
+F 1 "D_Small" V 10305 4332 50  0000 R CNN
+F 2 "" V 10350 4400 50  0001 C CNN
+F 3 "~" V 10350 4400 50  0001 C CNN
+	1    10350 4400
+	0    -1   -1   0
+$EndComp
+Wire Wire Line
+	10350 4300 10550 4300
+Wire Wire Line
+	10100 3050 10100 3450
+Connection ~ 10100 3450
+Wire Wire Line
+	10100 3450 10100 4100
+Wire Wire Line
+	10750 3050 10750 3450
+Connection ~ 10750 3450
+Wire Wire Line
+	10750 3450 10750 4100
+Wire Wire Line
+	10350 3850 9700 3850
+Connection ~ 9700 3850
+Wire Wire Line
+	9700 3850 9400 3850
+Wire Wire Line
+	10350 4500 9700 4500
+Connection ~ 9700 4500
+Wire Wire Line
+	9700 4500 9400 4500
+Text GLabel 9400 3850 0    50   Input ~ 0
+ROW0
+Text GLabel 9400 4500 0    50   Input ~ 0
+ROW1
+Text GLabel 10100 3050 1    50   Input ~ 0
+COL0
+Text GLabel 10750 3050 1    50   Input ~ 0
+COL1
 $EndSCHEMATC

Commit message: Footprints Assigned
Parts:
- C1, C2, C3, C4, C5, C6, C7: renamed from C?; footprint (none) -> Capacitor_SMD:C_0805_2012Metric
- D1, D2, D3, D4: renamed from D?; footprint (none) -> Diode_SMD:D_SOD-123
- F1: renamed from F?; footprint (none) -> Fuse:Fuse_1206_3216Metric
- MX1, MX2, MX3, MX4: renamed from MX?; footprint (none) -> MX_Alps_Hybrid:MX-1.5U-NoLED
- R1, R2, R3, R4: renamed from R?; footprint (none) -> Resistor_SMD:R_0805_2012Metric
- SW1: renamed from SW?; footprint (none) -> random-keyboard-parts:SKQG-1155865
- USB1: renamed from USB?; footprint (none) -> random-keyboard-parts:Molex-0548190589
- Y1: renamed from Y?; footprint (none) -> Crystal:Crystal_SMD_3225-4Pin_3.2x2.5mm
- gave numbers to parts that had none: 1

Commit message: Finished PCB
Parts:
- MX1, MX2, MX3, MX4: footprint MX_Alps_Hybrid:MX-1.5U-NoLED -> MX_Alps_Hybrid:MX-1U-NoLED
Connections:
- net COL0: now also MX3.1 (COL); no longer MX2.1 (COL)
- net COL1: now also D1.1 (K), D2.1 (K), D4.2 (A), MX2.1 (COL), MX4.2 (ROW); no longer MX3.1 (COL)
- net ROW1: now also D3.1 (K); no longer D2.1 (K)
- removed net ROW0: D1.1 (K), D3.1 (K)
Other:
- moved on the sheet: D1, D2, D3, D4, MX1, MX2, MX3, MX4
Changed lines of the file:
@@
 L MX_Alps_Hybrid:MX-NoLED MX1
 U 1 1 63548E84
-P 9950 3500
-F 0 "MX1" H 9983 3723 60  0000 C CNN
-F 1 "MX-NoLED" H 9983 3649 20  0000 C CNN
-F 2 "MX_Alps_Hybrid:MX-1.5U-NoLED" H 9325 3475 60  0001 C CNN
-F 3 "" H 9325 3475 60  0001 C CNN
-	1    9950 3500
+P 9700 3500
+F 0 "MX1" H 9733 3723 60  0000 C CNN
+F 1 "MX-NoLED" H 9733 3649 20  0000 C CNN
+F 2 "MX_Alps_Hybrid:MX-1U-NoLED" H 9075 3475 60  0001 C CNN
+F 3 "" H 9075 3475 60  0001 C CNN
+	1    9700 3500
 	1    0    0    -1
 $EndComp
@@
 L Device:D_Small D1
 U 1 1 6354A380
-P 9700 3750
-F 0 "D1" V 9746 3682 50  0000 R CNN
-F 1 "D_Small" V 9655 3682 50  0000 R CNN
-F 2 "Diode_SMD:D_SOD-123" V 9700 3750 50  0001 C CNN
-F 3 "~" V 9700 3750 50  0001 C CNN
-	1    9700 3750
+P 9450 3750
+F 0 "D1" V 9496 3682 50  0000 R CNN
+F 1 "D_Small" V 9405 3682 50  0000 R CNN
+F 2 "Diode_SMD:D_SOD-123" V 9450 3750 50  0001 C CNN
+F 3 "~" V 9450 3750 50  0001 C CNN
+	1    9450 3750
 	0    -1   -1   0
 $EndComp
 Wire Wire Line
-	9700 3650 9900 3650
+	9450 3650 9650 3650
 $Comp
 L MX_Alps_Hybrid:MX-NoLED MX3
 U 1 1 63552C0D
-P 10600 3500
-F 0 "MX3" H 10633 3723 60  0000 C CNN
-F 1 "MX-NoLED" H 10633 3649 20  0000 C CNN
-F 2 "MX_Alps_Hybrid:MX-1.5U-NoLED" H 9975 3475 60  0001 C CNN
-F 3 "" H 9975 3475 60  0001 C CNN
-	1    10600 3500
+P 9700 4150
+F 0 "MX3" H 9733 4373 60  0000 C CNN
+F 1 "MX-NoLED" H 9733 4299 20  0000 C CNN
+F 2 "MX_Alps_Hybrid:MX-1U-NoLED" H 9075 4125 60  0001 C CNN
+F 3 "" H 9075 4125 60  0001 C CNN
+	1    9700 4150
 	1    0    0    -1
 $EndComp
@@
 L Device:D_Small D3
 U 1 1 63552C17
-P 10350 3750
-F 0 "D3" V 10396 3682 50  0000 R CNN
-F 1 "D_Small" V 10305 3682 50  0000 R CNN
-F 2 "Diode_SMD:D_SOD-123" V 10350 3750 50  0001 C CNN
-F 3 "~" V 10350 3750 50  0001 C CNN
-	1    10350 3750
+P 9450 4400
+F 0 "D3" V 9496 4332 50  0000 R CNN
+F 1 "D_Small" V 9405 4332 50  0000 R CNN
+F 2 "Diode_SMD:D_SOD-123" V 9450 4400 50  0001 C CNN
+F 3 "~" V 9450 4400 50  0001 C CNN
+	1    9450 4400
 	0    -1   -1   0
 $EndComp
 Wire Wire Line
-	10350 3650 10550 3650
+	9450 4300 9650 4300
 $Comp
 L MX_Alps_Hybrid:MX-NoLED MX2
 U 1 1 63556D1C
-P 9950 4150
-F 0 "MX2" H 9983 4373 60  0000 C CNN
-F 1 "MX-NoLED" H 9983 4299 20  0000 C CNN
-F 2 "MX_Alps_Hybrid:MX-1.5U-NoLED" H 9325 4125 60  0001 C CNN
-F 3 "" H 9325 4125 60  0001 C CNN
-	1    9950 4150
+P 10250 3500
+F 0 "MX2" H 10283 3723 60  0000 C CNN
+F 1 "MX-NoLED" H 10283 3649 20  0000 C CNN
+F 2 "MX_Alps_Hybrid:MX-1U-NoLED" H 9625 3475 60  0001 C CNN
+F 3 "" H 9625 3475 60  0001 C CNN
+	1    10250 3500
 	1    0    0    -1
 $EndComp
@@
 L Device:D_Small D2
 U 1 1 63556D26
-P 9700 4400
-F 0 "D2" V 9746 4332 50  0000 R CNN
-F 1 "D_Small" V 9655 4332 50  0000 R CNN
-F 2 "Diode_SMD:D_SOD-123" V 9700 4400 50  0001 C CNN
-F 3 "~" V 9700 4400 50  0001 C CNN
-	1    9700 4400
+P 10000 3750
+F 0 "D2" V 10046 3682 50  0000 R CNN
+F 1 "D_Small" V 9955 3682 50  0000 R CNN
+F 2 "Diode_SMD:D_SOD-123" V 10000 3750 50  0001 C CNN
+F 3 "~" V 10000 3750 50  0001 C CNN
+	1    10000 3750
 	0    -1   -1   0
 $EndComp
 Wire Wire Line
-	9700 4300 9900 4300
+	10000 3650 10200 3650
+Wire Wire Line
+	9850 3050 9850 3450
+Connection ~ 9850 3450
+Wire Wire Line
+	9850 3450 9850 4100
+Wire Wire Line
+	9450 3850 9150 3850
+Text GLabel 9150 3850 0    50   Input ~ 0
+ROW0
+Text GLabel 8500 4500 0    50   Input ~ 0
+ROW1
+Text GLabel 9850 3050 1    50   Input ~ 0
+COL0
+Text GLabel 10400 3050 1    50   Input ~ 0
+COL1
+Wire Wire Line
+	10400 3450 10400 3050
+Wire Wire Line
+	10000 4300 10200 4300
+$Comp
+L Device:D_Small D4
+U 1 1 63559CB0
+P 10000 4400
+F 0 "D4" V 10046 4332 50  0000 R CNN
+F 1 "D_Small" V 9955 4332 50  0000 R CNN
+F 2 "Diode_SMD:D_SOD-123" V 10000 4400 50  0001 C CNN
+F 3 "~" V 10000 4400 50  0001 C CNN
+	1    10000 4400
+	0    -1   -1   0
+$EndComp
 $Comp
 L MX_Alps_Hybrid:MX-NoLED MX4
 U 1 1 63559CA6
-P 10600 4150
-F 0 "MX4" H 10633 4373 60  0000 C CNN
-F 1 "MX-NoLED" H 10633 4299 20  0000 C CNN
-F 2 "MX_Alps_Hybrid:MX-1.5U-NoLED" H 9975 4125 60  0001 C CNN
-F 3 "" H 9975 4125 60  0001 C CNN
-	1    10600 4150
+P 10250 4150
+F 0 "MX4" H 10283 4373 60  0000 C CNN
+F 1 "MX-NoLED" H 10283 4299 20  0000 C CNN
+F 2 "MX_Alps_Hybrid:MX-1U-NoLED" H 9625 4125 60  0001 C CNN
+F 3 "" H 9625 4125 60  0001 C CNN
+	1    10250 4150
 	1    0    0    -1
 $EndComp
-$Comp
-L Device:D_Small D4
-U 1 1 63559CB0
-P 10350 4400
-F 0 "D4" V 10396 4332 50  0000 R CNN
-F 1 "D_Small" V 10305 4332 50  0000 R CNN
-F 2 "Diode_SMD:D_SOD-123" V 10350 4400 50  0001 C CNN
-F 3 "~" V 10350 4400 50  0001 C CNN
-	1    10350 4400
-	0    -1   -1   0
-$EndComp
+Connection ~ 9450 4500
 Wire Wire Line
-	10350 4300 10550 4300
+	9450 4500 10000 4500
 Wire Wire Line
-	10100 3050 10100 3450
-Connection ~ 10100 3450
+	8500 4500 9450 4500
 Wire Wire Line
-	10100 3450 10100 4100
+	10000 3850 10000 4300
+Connection ~ 10000 4300
 Wire Wire Line
-	10750 3050 10750 3450
-Connection ~ 10750 3450
+	10400 3450 10400 3850
+Connection ~ 10400 3450
 Wire Wire Line
-	10750 3450 10750 4100
+	9450 3850 10000 3850
+Connection ~ 9450 3850
+Connection ~ 10400 3850
 Wire Wire Line
-	10350 3850 9700 3850
-Connection ~ 9700 3850
+	10400 3850 10400 4100
+Connection ~ 10000 3850
 Wire Wire Line
-	9700 3850 9400 3850
-Wire Wire Line
-	10350 4500 9700 4500
-Connection ~ 9700 4500
-Wire Wire Line
-	9700 4500 9400 4500
-Text GLabel 9400 3850 0    50   Input ~ 0
-ROW0
-Text GLabel 9400 4500 0    50   Input ~ 0
-ROW1
-Text GLabel 10100 3050 1    50   Input ~ 0
-COL0
-Text GLabel 10750 3050 1    50   Input ~ 0
-COL1
+	10000 3850 10400 3850
 $EndSCHEMATC

Commit message: Actually Finished this time
Connections:
- net COL0: now also U1.29 (PB5)
- net COL1: now also U1.31 (PC6), U1.32 (PC7)
- net ROW1: now also U1.30 (PB6)
Changed lines of the file:
@@
 Wire Wire Line
 	10000 3850 10400 3850
+Text GLabel 6400 3400 2    50   Input ~ 0
+COL1
+Text GLabel 6400 2900 2    50   Input ~ 0
+COL0
+Text GLabel 6400 3300 2    50   Input ~ 0
+ROW0
+Text GLabel 6400 3000 2    50   Input ~ 0
+ROW1
 $EndSCHEMATC

Commit message: New Trace Layout
Connections:
- net COL0: now also U1.28 (PB4); no longer U1.29 (PB5)
- net COL1: now also U1.26 (PD6), U1.29 (PB5); no longer U1.31 (PC6), U1.32 (PC7)
- net ROW1: now also U1.27 (PD7); no longer U1.30 (PB6)
Changed lines of the file:
@@
 Wire Wire Line
 	10000 3850 10400 3850
-Text GLabel 6400 3400 2    50   Input ~ 0
+Text GLabel 6400 4200 2    50   Input ~ 0
 COL1
+Text GLabel 6400 2800 2    50   Input ~ 0
+COL0
 Text GLabel 6400 2900 2    50   Input ~ 0
-COL0
-Text GLabel 6400 3300 2    50   Input ~ 0
 ROW0
-Text GLabel 6400 3000 2    50   Input ~ 0
+Text GLabel 6400 4300 2    50   Input ~ 0
 ROW1
 $EndSCHEMATC
